File: SolarCamPiV2.kicad_sch (KiCad schematic)
At the start: 99 parts, among them J1 TagConnect_TC2030_SWD, J2 RPi, J3 FTDI_RPI, Q1 AO3401A, Q2 AO3401A, Q3 2N7002, Q4 AO3401A, Q5 2N7002, Q6 BSS84, SW1 User, U1 CN3767, U2 HT7533, U3 SY8113B, U4 STM32G031Fx, Y1 32.768kHz

Commit message: Add fabrication files
Parts:
- D3: LCSC (none) -> C68978
- J3: LCSC (none) -> C2935912
- JP1, JP4: LCSC (none) -> C2935927
Changed lines of the file:
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@@
+      (effects (font (size 1.27 1.27)) hide)
+    )
+    (property "LCSC" "C2935927" (id 4) (at 140.97 148.59 90)
       (effects (font (size 1.27 1.27)) hide)
     )
@@
     )
     (property "Datasheet" "~" (id 3) (at 158.75 148.59 0)
+      (effects (font (size 1.27 1.27)) hide)
+    )
+    (property "LCSC" "C2935927" (id 4) (at 158.75 148.59 90)
       (effects (font (size 1.27 1.27)) hide)
     )
@@
     )
     (property "Datasheet" "https://assets.nexperia.com/documents/data-sheet/BAV70_SER.pdf" (id 3) (at 209.55 71.12 0)
+      (effects (font (size 1.27 1.27)) hide)
+    )
+    (property "LCSC" "C68978" (id 4) (at 209.55 71.12 90)
       (effects (font (size 1.27 1.27)) hide)
     )
@@
       (effects (font (size 1.27 1.27)) hide)
     )
+    (property "LCSC" "C2935912" (id 4) (at 261.62 121.92 0)
+      (effects (font (size 1.27 1.27)) hide)
+    )
